File: Power.kicad_sch (KiCad schematic)
At the start: 50 parts, among them Q1 FDN86246, Q2 VOS617A-7T, T1 POE70P-50L, U1 TPS23753APW, U3 TLV431ACDBZR

Commit message: changed MOUSER# for R13 and arranged reference designators on PCB
Parts:
- R17: MOUSER# 603-RC0402FR-0713K3L -> 603-RC0402FR-0713K3P; MOUSER#.Var 3.3V(652-CR0402FX-2432GLF) 5V(603-RC0402FR-0713K3L) -> 3.3V(652-CR0402FX-2432GLF) 5V(603-RC0402FR-0713K3P)
Changed lines of the file:
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@@
 			)
 		)
-		(property "MOUSER#" "603-RC0402FR-0713K3L"
+		(property "MOUSER#" "603-RC0402FR-0713K3P"
 			(at 254 143.51 0)
 			(effects
@@
 			)
 		)
-		(property "MOUSER#.Var" "3.3V(652-CR0402FX-2432GLF) 5V(603-RC0402FR-0713K3L)"
+		(property "MOUSER#.Var" "3.3V(652-CR0402FX-2432GLF) 5V(603-RC0402FR-0713K3P)"
 			(at 254 143.51 0)
 			(effects
