File: Ethernet.kicad_sch (KiCad schematic)
At the start: 41 parts, among them T2 S558-5500-25-F, U4 LAN8720A, Y1 ECS-2333-500-BN-TR

Commit message: all parts geo-renamed
Parts:
- renumbered C24 to 1C3, C25 to 1C5, C34 to 1C9, D1 to 1D3, L2 to 1L2, R31 to 1R4, R27 to 1R5, T2 to 1T2, U4 to 1U1, C33 to 2C10, C31 to 2C12, C35 to 2C13, C32 to 2C14, C16 to 2C18, C53 to 2C19, C52 to 2C20, C54 to 2C21, C51 to 2C22, C27 to 2C24, C30 to 2C25, C26 to 2C27, C29 to 2C34, C28 to 2C39, R32 to 2R13, R30 to 2R15, R34 to 2R16, R33 to 2R17, R35 to 2R18, R29 to 2R19, R36 to 2R26, R37 to 2R27, R38 to 2R28, R19 to 2R29, R25 to 2R30, R24 to 2R31, R26 to 2R32, R23 to 2R33, R14 to 2R34, R22 to 2R35, R20 to 2R37, Y1 to 2Y1

Commit message: properties cleanup added unique parts ID
Parts:
- 1C3, 1C5: IDAnything (none) -> 9rwxvasa5ehn0bvjk789fvwtcg
- 1C9: IDAnything (none) -> e5kfcvbxymkwra6w8qtzj3bv2h
- 1D3: IDAnything (none) -> e9zh6hyq7ajky9a0s8vpv9p37r
- 1L2: IDAnything (none) -> 4a2ahq0xf2kzhaz1w3cmtsqf2g
- 1R4, 1R5, 2R16, 2R17, 2R18, 2R26, 2R27, 2R28: IDAnything (none) -> ftsp2a555thn6bt15g7x2jan0j
- 1T2: IDAnything (none) -> d31xqqjt10gnn9h61fg6gqtx78
- 1U1: IDAnything (none) -> 9b7k6rnvayhd6attwbw8g6npsh
- 2C10, 2C12, 2C14: IDAnything (none) -> bxzbaywtstgjdb4bw6yay3xr4b
- 2C13: IDAnything (none) -> 346tvkh6ytke3bys71dsn4g0r8
- 2C18: IDAnything (none) -> 5cec8xb21wkrn9jazn0tx4yt0k
- 2C19, 2C20, 2C21, 2C22: IDAnything (none) -> 9zm41knhygg4gbefdxyjca9sqq
- 2C25: IDAnything (none) -> cp71jb8htmjycabjvbztj9p7aw
- 2R13: IDAnything (none) -> ab87j4h0awjq682gnnp5ww3py5
- 2R15: IDAnything (none) -> c1vc3q1ecwg38aepd291cy2avj
- 2R19: IDAnything (none) -> a31vzph314kf585hmxr9m1ypj6
- 2R29, 2R34, 2R35, 2R37: IDAnything (none) -> 51rzmzs5b4j9y8fva05p13xw6s
- 2R30, 2R31, 2R32, 2R33: IDAnything (none) -> fr13wzhp50gkdbhgg77yeh5c2f
- 2Y1: IDAnything (none) -> cftj26szx4gzy8x6v5b860read

Commit message: added some LCSC part numbers
Parts:
- 1D3: LCSC# (none) -> C553132
- 1T2: LCSC# (none) -> C5373193
- 1U1: LCSC# (none) -> C45223
- 2Y1: LCSC# (none) -> C2848221
